File: keyboard pcb/Keyboard/Keyboard-Doomsday-Deck.kicad_pcb (KiCad board)
At the start: 2 copper layers, 194.5 x 130.5 mm, 105 parts, among them J1 Conn_01x05, J2 Conn_01x02, J3 Conn_01x02, J4 OLED, U1 Raspberry_Pi_Pico2

Commit message: ain
Parts:
- J4: footprint Connector_PinHeader_2.54mm:PinHeader_1x04_P2.54mm_Vertical -> ScottoKeebs_Components:OLED_128x32
- U1: moved to B.Cu
- moved J4 11.4 mm to (171.1, 40.0)
- moved U1 2.50 mm to (102.5, 155.0)
Connections:
- U1 pad 24: Net-(U1-GPIO18) -> unconnected-(U1-GPIO18-Pad24)_1
- U1 pad 25: Net-(U1-GPIO19) -> unconnected-(U1-GPIO19-Pad25)
- U1 pad 36: 3.3V -> +3.3V
- U1 pad 40: GND -> unconnected-(U1-VBUS-Pad40)
Routing:
- net 3.3V: track 263.2 -> 82.8 mm
- net JOY_Y: track 304.2 -> 139.6 mm
- net SDA: track 157.7 -> 222.1 mm
- net ROW1: track 398.3 -> 336.9 mm
- net ROW2: track 396.6 -> 341.9 mm
- net SCL: track 164.0 -> 218.5 mm
- net COL10: track 184.0 -> 229.7 mm, vias 0 -> 1
- net ROW3: track 353.2 -> 309.4 mm
- net JLEFT_CLICK: track 101.8 -> 142.2 mm
- net ROW4: track 458.4 -> 420.5 mm
- net COL9: track 167.5 -> 205.1 mm, vias 0 -> 1
- net COL8: track 154.1 -> 188.9 mm, vias 0 -> 1
- net COL6: track 149.0 -> 182.9 mm
- net ROW5: track 382.3 -> 350.4 mm
- net COL2: track 171.0 -> 193.5 mm
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Other:
- board text added: ":D"
- board text removed: "-TANMAY"
