File: keyboard pcb/Keyboard/Keyboard-Doomsday-Deck.kicad_sch (KiCad schematic)
At the start: 1 part, among them U1 Raspberry_Pi_Pico2

Commit message: ain
Connections:
- net 3.3V: no longer U1.36 (3V3)
- new net +3.3V: U1.36 (3V3)
