File: keyboard pcb/Keyboard/OLED_KEYBOARD.kicad_sch (KiCad schematic)
At the start: 1 part, among them J4 OLED

Commit message: ain
Parts:
- J4: footprint Connector_PinHeader_2.54mm:PinHeader_1x04_P2.54mm_Vertical -> ScottoKeebs_Components:OLED_128x32
Changed lines of the file:
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@@
 			)
 		)
-		(property "Footprint" "Connector_PinHeader_2.54mm:PinHeader_1x04_P2.54mm_Vertical"
+		(property "Footprint" "ScottoKeebs_Components:OLED_128x32"
 			(at 91.44 80.01 0)
 			(hide yes)
@@
 		)
 		(instances
-			(project "Keyboard-Zerodeck"
+			(project "Keyboard-Doomsday-Deck"
 				(path "/83b0bf1e-f042-47d2-8247-013ebbe736a1/a7003389-5ce7-40cf-8381-041682537b6d"
 					(reference "J4")
