File: carrier-orange pi zero 3w/USB.kicad_sch (KiCad schematic)
At the start: 17 parts, among them U2 USB2517I-JZX, Y1 24.000MHz

Commit message: Update Orange Pi carrier board
Parts:
- added J7: OPI_USB2_UPSTREAM, symbol Connector:Conn_01x05_Pin
- added R6, R7: 100 kΩ, symbol Device:R
Connections:
- net GND: now also J7.4 (Pin_4), R7.1
- net VBUS_DET: now reaches U2.44 (VBUS_DET)
- net VBUS_DET: now also R6.1, R7.2
- net OPI_USB_DM: now reaches U2.58 (USBUP_DM)
- net OPI_USB_DM: now also J7.3 (Pin_3)
- net OPI_USB_DP: now reaches U2.59 (USBUP_DP)
- net OPI_USB_DP: now also J7.2 (Pin_2)
- new net OPI_USB_CC: J7.5 (Pin_5)
- new net OPI_USB_VBUS: J7.1 (Pin_1), R6.2
- no-connect marks 2 -> 0
