File: carrier-orange pi zero 3w/USB.kicad_sch (KiCad schematic)
At the start: 46 parts, among them J8 USB_C_Receptacle_USB2.0_16P, Q1 Q_PMOS_GSD, Q2 2N7002, U2 USB2517I-JZX, U3 TPD2EUSB30DRTR, Y1 24.000MHz

Commit message: ain
Parts:
- C19, C21, C27: value 1 µF -> 1µF
- R11, R12, R13, R14, R15, R16, R17, R18, R19, R20, R21, R22, R23, R27, R28: value 10 kΩ -> 10k
- R24: value 100kΩ -> 100k
- R25: value 10kΩ -> 10k
- R26: value 100 kΩ -> 100k
- R4: value 1 MΩ -> 1M
- R5: value 12.0 kΩ -> 12.0k
- R8, R9: value 5.1 kΩ -> 5.1k
Changed lines of the file:
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@@
 			(effects
 				(font
-					(size 1.27 1.27)
+					(size 1.016 1.016)
 				)
 				(justify left)
@@
 			)
 		)
-		(property "Value" "10 kΩ"
-			(at 130.81 87.884 90)
+		(property "Value" "10k"
+			(at 130.81 87.63 90)
 			(show_name no)
 			(do_not_autoplace no)
@@
 			(effects
 				(font
-					(size 1.27 1.27)
+					(size 1.016 1.016)
 				)
 				(justify left)
@@
 			(effects
 				(font
-					(size 1.27 1.27)
+					(size 1.016 1.016)
 				)
 			)
@@
 			)
 		)
-		(property "Value" "10 kΩ"
+		(property "Value" "10k"
 			(at 196.85 29.21 90)
 			(show_name no)
@@
 		(in_pos_files yes)
 		(dnp no)
-		(fields_autoplaced yes)
 		(property "Reference" "R7"
-			(at 138.43 22.86 90)
+			(at 138.43 27.178 90)
 			(show_name no)
 			(do_not_autoplace no)
@@
 		)
 		(property "Value" "100k"
-			(at 138.43 25.4 90)
+			(at 138.43 29.21 90)
 			(show_name no)
 			(do_not_autoplace no)
 			(effects
 				(font
-					(size 1.27 1.27)
+					(size 1.016 1.016)
 				)
 			)
@@
 			)
 		)
-		(property "Value" "10 kΩ"
+		(property "Value" "10k"
 			(at 251.46 109.22 90)
 			(show_name no)
@@
 			)
 		)
-		(property "Value" "5.1 kΩ"
-			(at 109.474 22.098 90)
+		(property "Value" "5.1k"
+			(at 109.474 24.13 90)
 			(show_name no)
 			(do_not_autoplace no)
@@
 			)
 		)
-		(property "Value" "10 kΩ"
+		(property "Value" "10k"
 			(at 251.46 88.9 90)
 			(show_name no)
@@
 			(effects
 				(font
-					(size 1.27 1.27)
+					(size 1.016 1.016)
 				)
 				(justify left)
@@
 			)
 		)
-		(property "Value" "10 kΩ"
-			(at 144.78 87.884 90)
+		(property "Value" "10k"
+			(at 144.78 86.36 90)
 			(show_name no)
 			(do_not_autoplace no)
@@
 			)
 		)
-		(property "Value" "10 kΩ"
+		(property "Value" "10k"
 			(at 251.46 83.82 90)
 			(show_name no)
@@
 			)
 		)
-		(property "Value" "10 kΩ"
+		(property "Value" "10k"
 			(at 87.63 112.014 90)
 			(show_name no)
@@
 			)
 		)
-		(property "Value" "1 µF"
+		(property "Value" "1µF"
 			(at 262.636 25.4 0)
 			(show_name no)
@@
 			(effects
 				(font
-					(size 1.27 1.27)
+					(size 1.016 1.016)
 				)
 				(justify left)
@@
 		(in_pos_files yes)
 		(dnp no)
-		(fields_autoplaced yes)
 		(property "Reference" "R6"
-			(at 148.59 22.86 90)
+			(at 148.59 26.924 90)
 			(show_name no)
 			(do_not_autoplace no)
@@
 		)
 		(property "Value" "100k"
-			(at 148.59 25.4 90)
+			(at 148.59 29.21 90)
 			(show_name no)
 			(do_not_autoplace no)
 			(effects
 				(font
-					(size 1.27 1.27)
+					(size 1.016 1.016)
 				)
 			)
@@
 			)
 		)
-		(property "Value" "10kΩ"
+		(property "Value" "10k"
 			(at 34.29 90.17 90)
 			(show_name no)
@@
 			)
 		)
-		(property "Value" "10 kΩ"
+		(property "Value" "10k"
 			(at 196.85 25.4 90)
 			(show_name no)
@@
 			)
 		)
-		(property "Value" "100 kΩ"
+		(property "Value" "100k"
 			(at 34.29 93.98 90)
 			(show_name no)
@@
 			(effects
 				(font
-					(size 1.27 1.27)
+					(size 1.016 1.016)
 				)
 				(justify left)
@@
 			)
 		)
-		(property "Value" "10 kΩ"
+		(property "Value" "10k"
 			(at 251.46 93.98 90)
 			(show_name no)
@@
 			)
 		)
-		(property "Value" "12.0 kΩ"
-			(at 38.1 52.832 90)
+		(property "Value" "12.0k"
+			(at 38.1 50.8 90)
 			(show_name no)
 			(do_not_autoplace no)
@@
 			(effects
 				(font
-					(size 1.27 1.27)
+					(size 1.016 1.016)
 				)
 				(justify left)
@@
 			)
 		)
-		(property "Value" "100kΩ"
-			(at 55.88 75.184 90)
+		(property "Value" "100k"
+			(at 55.88 74.93 90)
 			(show_name no)
 			(do_not_autoplace no)
@@
 			)
 		)
-		(property "Value" "1 µF"
+		(property "Value" "1µF"
 			(at 237.49 49.53 90)
 			(show_name no)
@@
 			(effects
 				(font
-					(size 1.27 1.27)
+					(size 1.016 1.016)
 				)
 			)
@@
 			)
 		)
-		(property "Value" "10 kΩ"
+		(property "Value" "10k"
 			(at 196.85 21.59 90)
 			(show_name no)
@@
 			)
 		)
-		(property "Value" "10 kΩ"
+		(property "Value" "10k"
 			(at 172.466 77.47 90)
 			(show_name no)
@@
 			)
 		)
-		(property "Value" "10 kΩ"
+		(property "Value" "10k"
 			(at 251.46 114.3 90)
 			(show_name no)
@@
 			)
 		)
-		(property "Value" "5.1 kΩ"
-			(at 109.474 28.702 90)
+		(property "Value" "5.1k"
+			(at 109.474 26.67 90)
 			(show_name no)
 			(do_not_autoplace no)
@@
 			)
 		)
-		(property "Value" "1 MΩ"
-			(at 34.798 25.4 90)
+		(property "Value" "1M"
+			(at 31.75 25.4 90)
 			(show_name no)
 			(do_not_autoplace no)
 			(effects
 				(font
-					(size 1.27 1.27)
+					(size 1.016 1.016)
 				)
 			)
@@
 			)
 		)
-		(property "Value" "10 kΩ"
-			(at 157.48 87.884 90)
+		(property "Value" "10k"
+			(at 157.48 86.614 90)
 			(show_name no)
 			(do_not_autoplace no)
@@
 			(effects
 				(font
-					(size 1.27 1.27)
+					(size 1.016 1.016)
 				)
 			)
@@
 			)
 		)
-		(property "Value" "10 kΩ"
+		(property "Value" "10k"
 			(at 251.46 104.14 90)
 			(show_name no)
@@
 			)
 		)
-		(property "Value" "10 kΩ"
+		(property "Value" "10k"
 			(at 251.46 99.06 90)
 			(show_name no)
@@
 			)
 		)
-		(property "Value" "1 µF"
-			(at 224.028 25.4 0)
+		(property "Value" "1µF"
+			(at 225.806 25.4 0)
 			(show_name no)
 			(do_not_autoplace no)
 			(effects
 				(font
-					(size 1.27 1.27)
+					(size 1.016 1.016)
 				)
 				(justify left)
@@
 			(effects
 				(font
-					(size 1.27 1.27)
+					(size 1.016 1.016)
 				)
 				(justify left)
