File: carrier-orange pi zero 3w/USB.kicad_sch (KiCad schematic)
At the start: 46 parts, among them J8 USB_C_Receptacle_USB2.0_16P, Q1 Q_PMOS_GSD, Q2 2N7002, U2 USB2517I-JZX, U3 TPD2EUSB30DRTR, Y1 24.000MHz

Commit message: ain
Parts:
- J8: footprint (none) -> Connector:FanPinHeader_1x04_P2.54mm_Vertical
- Q1: footprint (none) -> Package_TO_SOT_SMD:SOT-23
- U2: footprint (none) -> USB2517I-JZX:QFN50P900X900X100-65N-D
- U3: footprint (none) -> footprints:DRT0003A
- Y1: footprint (none) -> Crystal:Crystal_SMD_3225-4Pin_3.2x2.5mm
Changed lines of the file:
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@@
 			)
 		)
-		(property "Footprint" ""
+		(property "Footprint" "footprints:DRT0003A"
 			(at 165.1 52.07 0)
 			(hide yes)
@@
 			)
 		)
-		(property "Footprint" ""
+		(property "Footprint" "Package_TO_SOT_SMD:SOT-23"
 			(at 62.23 88.9 0)
 			(hide yes)
@@
 			)
 		)
-		(property "Footprint" ""
+		(property "Footprint" "USB2517I-JZX:QFN50P900X900X100-65N-D"
 			(at 204.14 92.71 0)
 			(hide yes)
@@
 			)
 		)
-		(property "Footprint" ""
+		(property "Footprint" "Connector:FanPinHeader_1x04_P2.54mm_Vertical"
 			(at 91.44 34.29 0)
 			(hide yes)
@@
 			)
 		)
-		(property "Footprint" ""
+		(property "Footprint" "Crystal:Crystal_SMD_3225-4Pin_3.2x2.5mm"
 			(at 17.78 25.4 0)
 			(hide yes)

Commit message: ain
Parts:
- removed J8: USB_C_Receptacle_USB2.0_16P, Connector:FanPinHeader_1x04_P2.54mm_Vertical, symbol Connector:USB_C_Receptacle_USB2.0_16P
- removed R8, R9: 5.1k, Resistor_SMD:R_0805_2012Metric, symbol Device:R
- added J8: Usb-C receptable, Connector_PinHeader_2.54mm:PinHeader_1x04_P2.54mm_Vertical, symbol Connector_Generic:Conn_01x04
- C23: value 100nF -> 1µF
- C25, C26: value 33pF -> 15pF
- F2: value MF-R500 -> 2920L500/6GR; footprint Capacitor_SMD:C_1206_3216Metric -> Fuse:Fuse_2920_7451Metric
- R4: value 1M -> 1MΩ
- U2: footprint USB2517I-JZX:QFN50P900X900X100-65N-D -> Package_DFN_QFN:VQFN-64-1EP_9x9mm_P0.5mm_EP5.4x5.4mm_ThermalVias
- U3: footprint footprints:DRT0003A -> SOT-723:SOT-723
- Y1: footprint Crystal:Crystal_SMD_3225-4Pin_3.2x2.5mm -> Crystal:Crystal_SMD_2016-4Pin_2.0x1.6mm
Connections:
- net GND: now also J8.4 (Pin_4)
- net OPI_USB_DM: now also J8.2 (Pin_2)
- net OPI_USB_DP: now also J8.3 (Pin_3)
- net OPI_USB_VBUS: now also J8.1 (Pin_1)
- no-connect marks 19 -> 17
