File: carrier-orange pi zero 3w/carrier-orange pi zero 3w.kicad_pcb (KiCad board)
At the start: 2 copper layers, 13 parts, among them J3 Orange Pi Zero 3W - 40-Pin GP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, J4 Conn_01x04_Pin, J5 ORANGE_PI_POWER_CABLE, J6 5V_PERIPHERALS, U1 TPS54302DDCT

Commit message: ain
Parts:
- added Q2: 2N7002, Package_TO_SOT_SMD:SOT-23, F.Cu at (207.4, 113.5)
Connections:
- J3 pad 3: unconnected-(J3-Pin_3-Pad3) -> /SDA
- J3 pad 5: unconnected-(J3-Pin_5-Pad5) -> /SCL
- J5 pad 4: unconnected-(J5-Pin_4-Pad4) -> Net-(J5-Pin_4)
