File: carrier-orange pi zero 3w/carrier-orange pi zero 3w.kicad_pcb (KiCad board)
At the start: 2 copper layers, 68 parts, among them J10 USB_A - 4, J11 USB_A - 5, J3 Orange Pi Zero 3W - 40-Pin GP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, J4 Conn_01x04_Pin, J5 ORANGE_PI_POWER_CABLE, J6 5V_PERIPHERALS, J7 USB_A - 1, J9 USB_A - 3, Q2 2N7002, U1 TPS54302DDCT

Commit message: ain
Parts:
- added ?: , , F.Cu at (73.8, 54.5)
- added ?: , , F.Cu at (73.8, 77.5)
- added ?: , , F.Cu at (131.8, 77.4)
- added ?: , , F.Cu at (131.8, 54.5)
- added C29: 47 µF, Capacitor_SMD:C_0805_2012Metric, F.Cu at (125.6, 123.7)
- added C30: 100 nF, Capacitor_SMD:C_0805_2012Metric, F.Cu at (125.6, 126.7)
- added IC1: MAX98357AETE+T, MAX98357AETE+T:QFN50P300X300X80-17N, F.Cu at (146.4, 131.9)
- added IC2: MAX98357AETE+T, MAX98357AETE+T:QFN50P300X300X80-17N, F.Cu at (146.4, 137.2)
- added J1: EPAPER_HAT_B, Connector_PinHeader_2.54mm:PinHeader_1x04_P2.54mm_Vertical, F.Cu at (137.5, 91.7)
- added J12: USB_A - 6, Connector:FanPinHeader_1x04_P2.54mm_Vertical, F.Cu at (-68.0, 148.2)
- added J13: USB_A - 7, Connector:FanPinHeader_1x04_P2.54mm_Vertical, F.Cu at (131.4, 30.5)
- added J14: USB_A - 2, Connector:FanPinHeader_1x04_P2.54mm_Vertical, F.Cu at (87.4, 29.5)
- added J15: FAN1, Connector_JST:JST_XH_B2B-XH-A_1x02_P2.50mm_Vertical, F.Cu at (98.5, 114.5)
- added J16: FAN2, Connector_JST:JST_XH_B2B-XH-A_1x02_P2.50mm_Vertical, F.Cu at (98.8, 124.2)
- added J2: CORE1262_HF, Waveshare_Core1262:Core1262_HF, F.Cu at (-58.7, 171.3)
- added J8: USB_C_Receptacle_USB2.0_16P, Connector:FanPinHeader_1x04_P2.54mm_Vertical, F.Cu at (65.4, 29.5)
- added Q1: Q_PMOS_GSD, Package_TO_SOT_SMD:SOT-23, F.Cu at (80.5, 161.5)
- added Q3: AO3400A, Package_TO_SOT_SMD:SOT-23, F.Cu at (125.8, 115.5)
- added Q4: AO3400A, Package_TO_SOT_SMD:SOT-23, F.Cu at (125.8, 119.9)
- added R29: 10K, Resistor_SMD:R_0805_2012Metric, F.Cu at (83.2, 138.5)
- added R30: 100K, Resistor_SMD:R_0805_2012Metric, F.Cu at (121.2, 114.7)
- added R31: 100, Resistor_SMD:R_0805_2012Metric, F.Cu at (121.2, 117.7)
- added R32: 100, Resistor_SMD:R_0805_2012Metric, F.Cu at (121.2, 120.6)
- added R33: 100K, Resistor_SMD:R_0805_2012Metric, F.Cu at (121.2, 123.6)
- added U2: USB2517I-JZX, USB2517I-JZX:QFN50P900X900X100-65N-D, F.Cu at (108.5, 98.5)
- added U3: TPD2EUSB30DRTR, footprints:DRT0003A, F.Cu at (122.9, 133.7)
- added Y1: 24.000MHz, Crystal:Crystal_SMD_3225-4Pin_3.2x2.5mm, F.Cu at (73.5, 154.5)
- J3: moved to B.Cu
- moved C10 155.9 mm to (-42.0, 148.9)
- moved J3 100.0 mm to (126.8, 55.5), turned to 90 degrees
- moved C1 90.5 mm to (24.5, 116.4)
- moved C11 90.5 mm to (29.5, 129.8)
- moved C12 90.5 mm to (29.5, 133.1)
- moved C13 90.5 mm to (48.9, 116.4)
- moved C14 90.5 mm to (48.9, 119.4)
- moved C15 90.5 mm to (42.1, 93.7)
- moved C16 90.5 mm to (42.1, 96.7)
- moved C17 90.5 mm to (42.1, 99.8)
- moved C18 90.5 mm to (42.1, 102.8)
- moved C19 90.5 mm to (42.1, 105.8)
- moved C2 90.5 mm to (24.5, 119.4)
- moved C20 90.5 mm to (46.5, 93.7)
- moved C21 90.5 mm to (46.5, 96.7)
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Connections:
- J3 pad 33: unconnected-(J3-Pin_33-Pad33) -> FAN1_PWM
- J3 pad 37: unconnected-(J3-Pin_37-Pad37) -> FAN2_PWM
Other:
- board text added: "3V3"
- board text added: "BUSY"
- board text added: "CLK"
- board text added: "CS"
- board text added: "DIO1"
- board text added: "DIO2"
- board text added: "MISO"
- board text added: "MOSI"
- board text added: "RESET"
- board text added: "RXEN"
- board text added: "TXEN"

Commit message: ain
Parts:
- removed IC1, IC2: MAX98357AETE+T, MAX98357AETE+T:QFN50P300X300X80-17N
- removed R29: 10K, Resistor_SMD:R_0805_2012Metric
- removed R8, R9: 5.1k, Resistor_SMD:R_0805_2012Metric
- added C31: 10µF, Capacitor_SMD:C_0805_2012Metric, F.Cu at (190.1, 107.7)
- added C32: 100nF, Capacitor_SMD:C_0805_2012Metric, F.Cu at (190.1, 110.7)
- added C33: 100nF, Capacitor_SMD:C_0805_2012Metric, F.Cu at (190.1, 113.7)
- added C34: 10µF, Capacitor_SMD:C_0805_2012Metric, F.Cu at (190.1, 116.7)
- added C35: 100nF, Capacitor_SMD:C_0805_2012Metric, F.Cu at (156.3, 114.1)
- added C36: 100µF, Capacitor_SMD:C_0805_2012Metric, F.Cu at (190.1, 119.7)
- added F3: 0.75A, Fuse:Fuse_1206_3216Metric, F.Cu at (111.3, 156.3)
- added F4: 1.5A, Fuse:Fuse_1812_4532Metric, F.Cu at (186.0, 103.7)
- added J17: L-SPEAKER, Connector_JST:JST_XH_B2B-XH-A_1x02_P2.50mm_Vertical, F.Cu at (176.6, 104.6)
- added J18: R-SPEAKER, Connector_JST:JST_XH_B2B-XH-A_1x02_P2.50mm_Vertical, F.Cu at (176.6, 112.4)
- added L1: 6.8uH, Inductor_SMD:L_Sunlord_SWPA8040S, F.Cu at (156.1, 148.8)
- added R34: 210k, Resistor_SMD:R_0805_2012Metric, F.Cu at (184.8, 118.3)
- added U4: L-MAX98357AETE+T, MAX98357AETE+T:QFN50P300X300X80-17N, F.Cu at (185.2, 108.8)
- added U5: R-MAX98357AETE+T, MAX98357AETE+T:QFN50P300X300X80-17N, F.Cu at (185.2, 114.2)
- added U7: MCP23017x-x-SO, Package_SO:SOIC-28W_7.5x17.9mm_P1.27mm, F.Cu at (147.6, 122.5)
- C23: value 100nF -> 1µF
- C25, C26: value 33pF -> 15pF
- C29: value 47 µF -> 47µF
- C30: value 100 nF -> 100nF
- F2: value MF-R500 -> 2920L500/6GR; footprint Capacitor_SMD:C_1206_3216Metric -> Fuse:Fuse_2920_7451Metric
- J1: footprint Connector_PinHeader_2.54mm:PinHeader_1x04_P2.54mm_Vertical -> Connector_PinHeader_2.54mm:PinHeader_1x08_P2.54mm_Vertical
- J5: value ORANGE_PI_POWER_CABLE -> Conn_01x20; footprint Connector_PinHeader_1.00mm:PinHeader_1x04_P1.00mm_Vertical -> Connector_FFC-FPC:TE_2-84952-0_1x20-1MP_P1.0mm_Horizontal
- J6: value 5V_PERIPHERALS -> PWR FOR DISPLAY
- J8: value USB_C_Receptacle_USB2.0_16P -> Usb-C receptable; footprint Connector:FanPinHeader_1x04_P2.54mm_Vertical -> Connector_PinHeader_2.54mm:PinHeader_1x04_P2.54mm_Vertical
- R1: value 10K -> 10k
- R4: value 1M -> 1MΩ
- U3: footprint footprints:DRT0003A -> SOT-723:SOT-723
- Y1: footprint Crystal:Crystal_SMD_3225-4Pin_3.2x2.5mm -> Crystal:Crystal_SMD_2016-4Pin_2.0x1.6mm
- moved J2 240.8 mm to (180.6, 145.0)
- moved J12 210.8 mm to (129.3, 74.0)
- moved C10 185.4 mm to (143.4, 153.7)
- moved J3 147.4 mm to (211.1, -65.4)
- moved ? 147.4 mm to (158.1, -66.5)
- moved ? 147.4 mm to (158.1, -43.5)
- moved ? 147.4 mm to (216.1, -43.5)
- moved ? 147.4 mm to (216.1, -66.4)
- moved J4 147.4 mm to (51.1, -90.7)
- moved C13 140.8 mm to (182.4, 71.8)
- moved C14 140.8 mm to (182.4, 74.8)
- moved R2 130.8 mm to (163.2, 152.6)
- moved R3 130.8 mm to (163.2, 155.6)
- moved R24 129.6 mm to (156.6, 71.7)
- moved F2 127.4 mm to (168.5, 88.8)
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Connections:
- J3 pad 11: unconnected-(J3-Pin_11-Pad11) -> UART_TX
- J3 pad 12: unconnected-(J3-Pin_12-Pad12) -> I2S_BCLK
- J3 pad 13: unconnected-(J3-Pin_13-Pad13) -> UART_RX
- J3 pad 2: unconnected-(J3-Pin_2-Pad2) -> +5V_OPI
- J3 pad 22: unconnected-(J3-Pin_22-Pad22) -> BUSY
- J3 pad 3: /SDA -> SDA
- J3 pad 35: unconnected-(J3-Pin_35-Pad35) -> I2S_LRCLK
- J3 pad 38: BUSY -> I2S_DIN
- J3 pad 4: unconnected-(J3-Pin_4-Pad4) -> +5V_OPI
- J3 pad 40: unconnected-(J3-Pin_40-Pad40) -> MCP_INT
- J3 pad 5: /SCL -> SCL
- J3 pad 6: unconnected-(J3-Pin_6-Pad6) -> GND
- J3 pad 7: unconnected-(J3-Pin_7-Pad7) -> SPI_CS_EXT
- J3 pad 9: unconnected-(J3-Pin_9-Pad9) -> GND
- J4 pad 2: /SCL -> SCL
- J4 pad 3: /SDA -> SDA
- J5 pad 1: +5V_OPI -> +5V_MAIN
- J5 pad 3: /power/CC -> +3V3_MAIN
- J5 pad 4: Net-(J5-Pin_4) -> GND
- J8 pad 1: (no net) -> OPI_USB_VBUS
- J8 pad 2: (no net) -> OPI_USB_DM
- J8 pad 3: (no net) -> OPI_USB_DP
- J8 pad 4: (no net) -> GND
- R1 pad 1: /power/CC -> +3V3_MAIN
- R1 pad 2: +5V_OPI -> Net-(U7-~{RESET})
Other:
- board text removed: "3V3"
- board text removed: "BUSY"
- board text removed: "CLK"
- board text removed: "CS"
- board text removed: "DIO1"
- board text removed: "DIO2"
- board text removed: "MISO"
- board text removed: "MOSI"
- board text removed: "RESET"
- board text removed: "RXEN"
- board text removed: "TXEN"

Commit message: ain
Parts:
- added J19: EXT-GPIO (BACKUP), Connector_PinHeader_2.54mm:PinHeader_2x10_P2.54mm_Vertical, F.Cu at (65.0, 99.8)
- C36: footprint Capacitor_SMD:C_0805_2012Metric -> Capacitor_SMD:CP_Elec_6.3x7.7
- J12: value USB_A - 6 -> USB_A - 6 (For Display)
- J13: value USB_A - 7 -> USB_A - 7 (For RTL SDR)
- J14: value USB_A - 2 -> USB_A - 2 (Extra/For phone )
- J15, J16, J17, J18: footprint Connector_JST:JST_XH_B2B-XH-A_1x02_P2.50mm_Vertical -> Connector_JST:JST_VH_B2P-VH_1x02_P3.96mm_Vertical
- J5: value Conn_01x20 -> EXT-GPIO
- U2: footprint USB2517I-JZX:QFN50P900X900X100-65N-D -> Package_DFN_QFN:VQFN-64-1EP_9x9mm_P0.5mm_EP5.4x5.4mm_ThermalVias
- moved J16 135.0 mm to (234.0, 92.7)
- moved J5 125.4 mm to (30.9, 113.0), turned to -90 degrees
- moved J15 120.0 mm to (220.7, 91.7)
- moved U7 105.9 mm to (47.2, 88.8)
- moved F3 100.3 mm to (194.4, 100.2)
- moved C29 86.8 mm to (189.4, 100.0)
- moved C30 86.8 mm to (189.4, 103.0)
- moved Q3 72.3 mm to (184.7, 100.7)
- moved R30 72.3 mm to (180.0, 100.0)
- moved R32 72.3 mm to (180.0, 105.9)
- moved Q4 72.3 mm to (184.7, 105.2)
- moved R31 72.3 mm to (180.0, 102.9)
- moved R33 72.3 mm to (180.0, 108.8)
- moved C1 47.1 mm to (152.4, 89.5)
- moved C10 47.1 mm to (152.4, 107.5)
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Connections:
- J12 pad 1: +5V_USB -> +5V_MAIN

Commit message: ain
Parts:
- J10, J11, J7, J9: footprint USB_A_4UCON_18666_KICAD10:USB_A_4UCON_18666 -> Connector_USB:USB_A_Molex_48037-2200_Horizontal
- J12, J13, J14: footprint Connector:FanPinHeader_1x04_P2.54mm_Vertical -> Connector_Phoenix_GMSTB:PhoenixContact_GMSTBA_2,5_4-G-7,62_1x04_P7.62mm_Horizontal
- J3: moved to F.Cu
- J4: moved to B.Cu
- moved Q1 291.8 mm to (-118.3, 150.1)
- moved Q2 291.8 mm to (-118.3, 154.5)
- moved C24 281.7 mm to (-100.1, 133.8)
- moved R19 281.7 mm to (-113.4, 124.7)
- moved R21 281.7 mm to (-113.4, 130.6)
- moved R25 281.7 mm to (-109.0, 124.7)
- moved R27 281.7 mm to (-109.0, 130.6)
- moved U3 281.7 mm to (-100.7, 147.4)
- moved Y1 281.7 mm to (-100.1, 144.1)
- moved C15 281.7 mm to (-104.5, 121.7)
- moved C19 281.7 mm to (-104.5, 133.8)
- moved C20 281.7 mm to (-100.1, 121.7)
- moved C21 281.7 mm to (-100.1, 124.7)
- moved C22 281.7 mm to (-100.1, 127.8)
- moved C23 281.7 mm to (-100.1, 130.8)
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Other:
- board outline added: 190 x 61 mm
- board text added: "+5V_OPI"
- board text added: "3v3"
- board text added: "BUSY"
- board text added: "DIO1"
- board text added: "EPAPER_BUSY"
- board text added: "EPAPER_CS"
- board text added: "EPAPER_DC"
- board text added: "EPAPER_RST"
- board text added: "FAN1_PWM"
- board text added: "FAN2_PWM"
- board text added: "GND-x"
- board text added: "I2S_BCLK"
- board text added: "I2S_DIN"
- board text added: "I2S_LRCLK"
- board text added: "LORA_CS"
- board text added: "MCP_INT"
- board text added: "RESET"
- board text added: "RXEN"
- board text added: "SPI3_MISO"
- board text added: "SPI3_MOSI"
- board text added: "SPI3_SCK"
- board text added: "SPI_CS_EXT"
- board text added: "TXEN"
- board text added: "UART0_RX"
- board text added: "UART0_TX"
- board text added: "UART7_RX"
- board text added: "UART7_TX"
- board text added: "UART_RX"
- board text added: "UART_TX"
