File: carrier-orange pi zero 3w/carrier-orange pi zero 3w.kicad_pcb (KiCad board)
At the start: 4 copper layers, 190 x 61 mm, 106 parts, among them J1 EPAPER_HAT_B, J10 USB_A - 4, J11 USB_A - 5, J12 USB_A - 6 (For Display), J13 USB_A - 7 (For RTL SDR), J14 USB_A - 2 (Extra/For phone ), J15 FAN1, J16 FAN2, J17 L-SPEAKER, J18 R-SPEAKER, J19 EXT-GPIO (BACKUP), J2 CORE1262_HF, J3 Orange Pi Zero 3W - 40-Pin GP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, J4 Conn_01x04_Pin, J5 EXT-GPIO, J6 PWR FOR DISPLAY, J7 USB_A - 1, J8 Usb-C receptable, J9 USB_A - 3, Q1 Q_PMOS_GSD, Q2 2N7002, Q3 AO3400A, Q4 AO3400A, U1 TPS54302DDCT, U2 USB2517I-JZX, U3 TPD2EUSB30DRTR, U4 L-MAX98357AETE+T, U5 R-MAX98357AETE+T, U7 MCP23017x-x-SO, Y1 24.000MHz

Commit message: ain
Parts:
- added R19: 10k, Resistor_SMD:R_0805_2012Metric, F.Cu at (116.5, 65.0)
- moved F4 4.65 mm to (143.4, 87.2)
- moved J19 1.98 mm to (99.5, 87.0)
- moved C6 1.91 mm to (170.7, 87.8)
- moved J15 1.76 mm to (64.2, 68.2)
- moved J17 1.64 mm to (64.1, 56.3)
- moved J6 1.35 mm to (177.7, 87.5)
- moved L1 1.35 mm to (136.0, 60.9)
- moved C33 0.78 mm to (233.9, 62.6)
- moved C34 0.78 mm to (235.9, 62.6)
Routing:
- net SPI3_MISO: track 33.0 -> 286.5 mm
- net SPI3_MOSI : track 36.2 -> 281.4 mm, vias 0 -> 4
- net SPI3_SCK: track 35.9 -> 271.3 mm, vias 0 -> 4
- net +3V3_MAIN: track 159.2 -> 358.9 mm, vias 11 -> 20
- net /USB/USB6DM: track 0.00 -> 199.6 mm, vias 0 -> 2
- net I2S_BCLK: track 0.00 -> 194.0 mm, vias 0 -> 2
- net /USB/USB7DM: track 0.00 -> 187.1 mm, vias 0 -> 2
- net /USB/USB7DP: track 0.00 -> 176.5 mm, vias 0 -> 1
- net MCP_INT: track 0.00 -> 175.9 mm, vias 0 -> 1
- net /USB/USB6DP: track 0.00 -> 163.1 mm, vias 0 -> 2
- net SPI_CS_EXT: track 32.8 -> 192.0 mm, vias 0 -> 2
- net I2S_DIN: track 35.3 -> 194.2 mm, vias 0 -> 3
- net I2S_LRCLK: track 43.7 -> 194.8 mm, vias 0 -> 1
- net UART_TX: track 35.6 -> 183.1 mm, vias 0 -> 3
- net UART_RX: track 32.5 -> 176.9 mm, vias 0 -> 1
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Other:
- board text added: "+"
- board text added: "+5"
- board text added: "-"
- board text added: "-(F1_SW)"
- board text added: "-(F2_SW)"
- board text added: "3V"
- board text added: "3V3"
- board text added: "5v"
- board text added: "D+"
- board text added: "D-"
- board text added: "GPIO1"
- board text added: "GPIO_2"
- board text added: "GPIO_3"
- board text added: "GPIO_4"
- board text added: "GPIO_5/INT"
- board text added: "GPIO_6/INT"
- board text added: "SPI_CS"

Commit message: ain
Parts:
- added G***: LOGO, LOGO, F.Cu at (207.0, 74.6)
- moved J2 6.27 mm to (229.0, 72.4)
- moved C33 3.67 mm to (233.4, 58.9)
- moved C34 3.67 mm to (235.4, 59.0)
- moved R34 3.56 mm to (230.2, 55.6)
- moved U5 2.99 mm to (234.2, 55.0)
Routing:
- net /USB/PRT_SWP6: track 130.2 -> 68.8 mm, vias 0 -> 2
- net /USB/USB6DM: track 199.6 -> 165.6 mm, vias 2 -> 3
- net GND: track 142.8 -> 117.0 mm, vias 72 -> 74
- net SPI3_MOSI : track 281.4 -> 269.4 mm, vias 4 -> 5
- net DIO1: track 90.8 -> 83.7 mm
- net MCP_INT: track 175.9 -> 182.7 mm
- net BUSY: track 71.0 -> 65.6 mm
- net SPI3_MISO: track 286.5 -> 283.1 mm
- net RESET: track 41.6 -> 38.2 mm
- net LORA_CS: track 55.8 -> 52.4 mm
- net +5V_FAN: track 248.9 -> 245.7 mm
- net RXEN: track 67.9 -> 65.2 mm
- net TXEN: track 60.4 -> 58.1 mm
- net +5V_AUDIO: track 227.5 -> 229.7 mm
- net +3V3_MAIN: track 358.9 -> 356.8 mm, vias 20 -> 18
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Other:
- outline, holes or cut-outs redrawn
- board text added: "O+"
