File: carrier-orange pi zero 3w/power.kicad_sch (KiCad schematic)
At the start: 22 parts, among them J4 Conn_01x04_Pin, J5 ORANGE_PI_POWER_CABLE, J6 5V_PERIPHERALS, U1 TPS54302DDCT

Commit message: ain
Parts:
- R29: footprint (none) -> Resistor_SMD:R_0805_2012Metric
Changed lines of the file:
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@@
 			)
 		)
-		(property "Footprint" ""
+		(property "Footprint" "Resistor_SMD:R_0805_2012Metric"
 			(at 48.26 114.808 90)
 			(hide yes)

Commit message: ain
Parts:
- removed J5: ORANGE_PI_POWER_CABLE, Connector_PinHeader_1.00mm:PinHeader_1x04_P1.00mm_Vertical, symbol Connector:Conn_01x04_Pin
- removed R1, R29: 10K, Resistor_SMD:R_0805_2012Metric, symbol Device:R
- J6: value 5V_PERIPHERALS -> PWR FOR DISPLAY
- L1: footprint (none) -> Inductor_SMD:L_Sunlord_SWPA8040S
Other:
- moved on the sheet: C4, C5, C6, F1

Commit message: ain
Parts:
- added F5: 3A, Fuse:Fuse_1812_4532Metric, symbol Device:Polyfuse
Connections:
- net +5V_MAIN: now also F5.1; no longer C2.1, C3.1, C7.1, J6.1 (Pin_1)
- new net +5V_PERIPH: C2.1, C3.1, C7.1, F5.2, J6.1 (Pin_1)
Changed lines of the file:
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@@
 	(wire
 		(pts
-			(xy 207.01 81.28) (xy 226.06 81.28)
+			(xy 207.01 81.28) (xy 212.09 81.28)
 		)
 		(stroke
@@
 		(pts
 			(xy 240.03 63.5) (xy 254 63.5)
+		)
+		(stroke
+			(width 0)
+			(type default)
+		)
+	)
+	(wire
+		(pts
+			(xy 219.71 81.28) (xy 226.06 81.28)
 		)
 		(stroke
@@
 					(unit 1)
 				)
+			)
+		)
+	)
+	(symbol
+		(lib_id "Device:Polyfuse")
+		(at 215.9 81.28 90)
+		(unit 1)
+		(body_style 1)
+		(exclude_from_sim no)
+		(in_bom yes)
+		(on_board yes)
+		(in_pos_files yes)
+		(dnp no)
+		(property "Reference" "F5"
+			(at 216.154 76.962 90)
+			(show_name no)
+			(do_not_autoplace no)
+			(effects
+				(font
+					(size 1.27 1.27)
+				)
+			)
+		)
+		(property "Value" "3A"
+			(at 215.9 79.248 90)
+			(show_name no)
+			(do_not_autoplace no)
+			(effects
+				(font
+					(size 1.27 1.27)
+				)
+			)
+		)
+		(property "Footprint" "Fuse:Fuse_1812_4532Metric"
+			(at 220.98 80.01 0)
+			(hide yes)
+			(show_name no)
+			(do_not_autoplace no)
+			(effects
+				(font
+					(size 1.27 1.27)
+				)
+				(justify left)
+			)
+		)
+		(property "Datasheet" ""
+			(at 215.9 81.28 0)
+			(hide yes)
+			(show_name no)
+			(do_not_autoplace no)
+			(effects
+				(font
+					(size 1.27 1.27)
+				)
+			)
+		)
+		(property "Description" "Resettable fuse, polymeric positive temperature coefficient"
+			(at 215.9 81.28 0)
+			(hide yes)
+			(show_name no)
+			(do_not_autoplace no)
+			(effects
+				(font
+					(size 1.27 1.27)
+				)
+			)
+		)
+		(pin "2"
+		)
+		(pin "1"
+		)
+		(instances
+			(project "carrier-orange pi zero 3w"
+				(path "/eed97ac6-b1d8-4052-bc40-1c993c6f2bcf/8a71e92a-c7a9-48a2-b776-d1fe91c6fc6f"
+					(reference "F5")
+					(unit 1)
+				)
