File: carrier-orange pi zero 3w/EINK.kicad_sch (KiCad schematic)
At the start: 3 parts, among them J1 EPAPER_HAT_B

Commit message: ain
Parts:
- J1: footprint (none) -> Connector_PinHeader_2.54mm:PinHeader_1x08_P2.54mm_Vertical
Changed lines of the file:
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@@
 			)
 		)
-		(property "Footprint" ""
+		(property "Footprint" "Connector_PinHeader_2.54mm:PinHeader_1x08_P2.54mm_Vertical"
 			(at 111.76 71.12 0)
 			(hide yes)
