File: carrier-orange pi zero 3w/EXTERNAL-GPIO.kicad_sch (KiCad schematic)
At the start: 5 parts, among them J19 EXT-GPIO (BACKUP), J5 EXT-GPIO, U7 MCP23017x-x-SO

Commit message: ain
Connections:
- no-connect marks 0 -> 11
Changed lines of the file:
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@@
 		(color 0 0 0 0)
 	)
+	(junction
+		(at 171.45 49.53)
+		(diameter 0)
+		(color 0 0 0 0)
+	)
+	(no_connect
+		(at 184.15 86.36)
+	)
+	(no_connect
+		(at 184.15 71.12)
+	)
+	(no_connect
+		(at 184.15 96.52)
+	)
+	(no_connect
+		(at 184.15 78.74)
+	)
+	(no_connect
+		(at 184.15 81.28)
+	)
+	(no_connect
+		(at 184.15 83.82)
+	)
+	(no_connect
+		(at 184.15 73.66)
+	)
+	(no_connect
+		(at 184.15 88.9)
+	)
+	(no_connect
+		(at 158.75 73.66)
+	)
+	(no_connect
+		(at 184.15 93.98)
+	)
+	(no_connect
+		(at 184.15 91.44)
+	)
 	(wire
 		(pts
@@
 	(wire
 		(pts
+			(xy 171.45 49.53) (xy 171.45 50.8)
+		)
+		(stroke
+			(width 0)
+			(type default)
+		)
+	)
+	(wire
+		(pts
 			(xy 171.45 101.6) (xy 171.45 104.14)
 		)
@@
 	(wire
 		(pts
-			(xy 171.45 44.45) (xy 171.45 50.8)
+			(xy 171.45 44.45) (xy 171.45 49.53)
 		)
 		(stroke
@@
 					(unit 1)
 				)
+			)
+		)
+	)
+	(symbol
+		(lib_id "power:PWR_FLAG")
+		(at 171.45 49.53 90)
+		(unit 1)
+		(body_style 1)
+		(exclude_from_sim no)
+		(in_bom yes)
+		(on_board yes)
+		(in_pos_files yes)
+		(dnp no)
+		(fields_autoplaced yes)
+		(property "Reference" "#FLG03"
+			(at 169.545 49.53 0)
+			(hide yes)
+			(show_name no)
+			(do_not_autoplace no)
+			(effects
+				(font
+					(size 1.27 1.27)
+				)
+			)
+		)
+		(property "Value" "PWR_FLAG"
+			(at 167.64 49.5299 90)
+			(show_name no)
+			(do_not_autoplace no)
+			(effects
+				(font
+					(size 1.27 1.27)
+				)
+				(justify left)
+			)
+		)
+		(property "Footprint" "Package_DIP:DIP-24_W7.62mm"
+			(at 171.45 49.53 0)
+			(hide yes)
+			(show_name no)
+			(do_not_autoplace no)
+			(effects
+				(font
+					(size 1.27 1.27)
+				)
+			)
+		)
+		(property "Datasheet" ""
+			(at 171.45 49.53 0)
+			(hide yes)
+			(show_name no)
+			(do_not_autoplace no)
+			(effects
+				(font
+					(size 1.27 1.27)
+				)
+			)
+		)
+		(property "Description" "Special symbol for telling ERC where power comes from"
+			(at 171.45 49.53 0)
+			(hide yes)
+			(show_name no)
+			(do_not_autoplace no)
+			(effects
+				(font
+					(size 1.27 1.27)
+				)
+			)
+		)
+		(pin "1"
+		)
+		(instances
+			(project "carrier-orange pi zero 3w"
+				(path "/eed97ac6-b1d8-4052-bc40-1c993c6f2bcf/a987d4c5-8c97-44d7-8286-7368f9e384c3"
+					(reference "#FLG03")
+					(unit 1)
+				)
