File: carrier-orange pi zero 3w/USB1-7.kicad_sch (KiCad schematic)
At the start: 7 parts, among them J10 USB_A - 4, J11 USB_A - 5, J12 USB_A - 6, J13 USB_A - 7, J14 USB_A - 2, J7 USB_A - 1, J9 USB_A - 3

Commit message: ain
Parts:
- J12, J13, J14: footprint (none) -> Connector:FanPinHeader_1x04_P2.54mm_Vertical
Changed lines of the file:
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@@
 			)
 		)
-		(property "Footprint" ""
+		(property "Footprint" "Connector:FanPinHeader_1x04_P2.54mm_Vertical"
 			(at 74.93 99.06 0)
 			(hide yes)
@@
 			)
 		)
-		(property "Footprint" ""
+		(property "Footprint" "Connector:FanPinHeader_1x04_P2.54mm_Vertical"
 			(at 73.66 128.27 0)
 			(hide yes)
@@
 			)
 		)
-		(property "Footprint" ""
+		(property "Footprint" "Connector:FanPinHeader_1x04_P2.54mm_Vertical"
 			(at 43.18 99.06 0)
 			(hide yes)

Commit message: ain
Parts:
- J12: value USB_A - 6 -> USB_A - 6 (For Display)
- J13: value USB_A - 7 -> USB_A - 7 (For RTL SDR)
- J14: value USB_A - 2 -> USB_A - 2 (Extra/For phone )
Connections:
- net +5V_USB: no longer J12.1 (VBUS)
- new net +5V_PERIPH: J12.1 (VBUS)
Changed lines of the file:
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@@
+		)
+	)
+	(wire
+		(pts
+			(xy 78.74 92.71) (xy 80.01 92.71)
+		)
+		(stroke
+			(width 0)
+			(type default)
 		)
 	)
@@
 	(global_label "+5V_USB"
 		(shape input)
-		(at 78.74 92.71 0)
-		(fields_autoplaced yes)
-		(effects
-			(font
-				(size 1.016 1.016)
-			)
-			(justify left)
-		)
-		(property "Intersheetrefs" "${INTERSHEET_REFS}"
-			(at 88.0464 92.71 0)
-			(hide yes)
-			(show_name no)
-			(do_not_autoplace no)
-			(effects
-				(font
-					(size 1.27 1.27)
-				)
-				(justify left)
-			)
-		)
-	)
-	(global_label "+5V_USB"
-		(shape input)
 		(at 80.01 63.5 0)
 		(fields_autoplaced yes)
@@
 		(property "Intersheetrefs" "${INTERSHEET_REFS}"
 			(at 56.2964 92.71 0)
+			(hide yes)
+			(show_name no)
+			(do_not_autoplace no)
+			(effects
+				(font
+					(size 1.27 1.27)
+				)
+				(justify left)
+			)
+		)
+	)
+	(global_label "+5V_PERIPH"
+		(shape input)
+		(at 80.01 92.71 0)
+		(fields_autoplaced yes)
+		(effects
+			(font
+				(size 1.27 1.27)
+			)
+			(justify left)
+		)
+		(property "Intersheetrefs" "${INTERSHEET_REFS}"
+			(at 94.7276 92.71 0)
 			(hide yes)
 			(show_name no)
@@
 			)
 		)
-		(property "Value" "USB_A - 6"
+		(property "Value" "USB_A - 6 (For Display)"
 			(at 71.12 87.63 0)
 			(show_name no)
@@
 			)
 		)
-		(property "Value" "USB_A - 7"
+		(property "Value" "USB_A - 7 (For RTL SDR)"
 			(at 69.85 116.84 0)
 			(show_name no)
@@
 			)
 		)
-		(property "Value" "USB_A - 2"
+		(property "Value" "USB_A - 2 (Extra/For phone )"
 			(at 39.37 87.63 0)
 			(show_name no)

Commit message: ain
Parts:
- J10, J11, J7, J9: footprint USB_A_4UCON_18666_KICAD10:USB_A_4UCON_18666 -> Connector_USB:USB_A_Molex_48037-2200_Horizontal
- J12, J13, J14: footprint Connector:FanPinHeader_1x04_P2.54mm_Vertical -> Connector_Phoenix_GMSTB:PhoenixContact_GMSTBA_2,5_4-G-7,62_1x04_P7.62mm_Horizontal
Connections:
- net GND: no longer J12.SH (Shield), J13.SH (Shield), J14.SH (Shield)

Commit message: ain
Parts:
- J12, J13, J14: footprint Connector_Phoenix_GMSTB:PhoenixContact_GMSTBA_2,5_4-G-7,62_1x04_P7.62mm_Horizontal -> Connector_PinHeader_2.54mm:PinHeader_1x04_P2.54mm_Vertical
Changed lines of the file:
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@@
 			)
 		)
-		(property "Footprint" "Connector_Phoenix_GMSTB:PhoenixContact_GMSTBA_2,5_4-G-7,62_1x04_P7.62mm_Horizontal"
+		(property "Footprint" "Connector_PinHeader_2.54mm:PinHeader_1x04_P2.54mm_Vertical"
 			(at 74.93 99.06 0)
 			(hide yes)
@@
 			)
 		)
-		(property "Footprint" "Connector_Phoenix_GMSTB:PhoenixContact_GMSTBA_2,5_4-G-7,62_1x04_P7.62mm_Horizontal"
+		(property "Footprint" "Connector_PinHeader_2.54mm:PinHeader_1x04_P2.54mm_Vertical"
 			(at 73.66 128.27 0)
 			(hide yes)
@@
 			)
 		)
-		(property "Footprint" "Connector_Phoenix_GMSTB:PhoenixContact_GMSTBA_2,5_4-G-7,62_1x04_P7.62mm_Horizontal"
+		(property "Footprint" "Connector_PinHeader_2.54mm:PinHeader_1x04_P2.54mm_Vertical"
 			(at 43.18 99.06 0)
 			(hide yes)
