File: carrier-orange pi zero 3w/carrier-orange pi zero 3w.kicad_sch (KiCad schematic)
At the start: 1 part, among them J3 Orange Pi Zero 3W - 40-Pin GP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

Commit message: ain
Other:
- moved on the sheet: J3

Commit message: ain
Connections:
- net BUSY: now also J3.22 (Pin_22); no longer J3.38 (Pin_38)
- net I2S_BCLK: now reaches J3.12 (Pin_12)
- net FAN1_PWM: now reaches J3.33 (Pin_33)
- net I2S_LRCLK: now reaches J3.35 (Pin_35)
- net FAN2_PWM: now reaches J3.37 (Pin_37)
- new net I2S_DIN: J3.38 (Pin_38)
- no-connect marks 25 -> 20
Other:
- added sheet AUDIO (Audio.kicad_sch)
- added sheet FAN (FAN.kicad_sch)

Commit message: ain
Connections:
- net UART_TX: now reaches J3.11 (Pin_11)
- net UART_RX: now reaches J3.13 (Pin_13)
- net +5V_OPI: now reaches J3.2 (Pin_2)
- net +5V_OPI: now also J3.4 (Pin_4)
- net MCP_INT: now reaches J3.40 (Pin_40)
- net GND: now reaches J3.6 (Pin_6)
- net GND: now also J3.9 (Pin_9)
- net SPI_CS_EXT: now reaches J3.7 (Pin_7)
- no-connect marks 20 -> 12
Other:
- added sheet EXTERNAL-GPIO (EXTERNAL-GPIO.kicad_sch)
- sheet power ports: added none; removed SCL, SDA

Commit message: ain
Connections:
- net GND: now also J3.25 (Pin_25)
- no-connect marks 12 -> 11
Changed lines of the file:
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@@
-	)
-	(no_connect
-		(at 139.7 101.6)
 	)
 	(no_connect
@@
 					(unit 1)
 				)
+			)
+		)
+	)
+	(symbol
+		(lib_id "power:GND")
+		(at 139.7 101.6 270)
+		(unit 1)
+		(body_style 1)
+		(exclude_from_sim no)
+		(in_bom yes)
+		(on_board yes)
+		(in_pos_files yes)
+		(dnp no)
+		(fields_autoplaced yes)
+		(property "Reference" "#PWR056"
+			(at 133.35 101.6 0)
+			(hide yes)
+			(show_name no)
+			(do_not_autoplace no)
+			(effects
+				(font
+					(size 1.27 1.27)
+				)
+			)
+		)
+		(property "Value" "GND"
+			(at 135.89 101.5999 90)
+			(show_name no)
+			(do_not_autoplace no)
+			(effects
+				(font
+					(size 1.27 1.27)
+				)
+				(justify right)
+			)
+		)
+		(property "Footprint" ""
+			(at 139.7 101.6 0)
+			(hide yes)
+			(show_name no)
+			(do_not_autoplace no)
+			(effects
+				(font
+					(size 1.27 1.27)
+				)
+			)
+		)
+		(property "Datasheet" ""
+			(at 139.7 101.6 0)
+			(hide yes)
+			(show_name no)
+			(do_not_autoplace no)
+			(effects
+				(font
+					(size 1.27 1.27)
+				)
+			)
+		)
+		(property "Description" "Power symbol creates a global label with name \"GND\" , ground"
+			(at 139.7 101.6 0)
+			(hide yes)
+			(show_name no)
+			(do_not_autoplace no)
+			(effects
+				(font
+					(size 1.27 1.27)
+				)
+			)
+		)
+		(pin "1"
+		)
+		(instances
+			(project "carrier-orange pi zero 3w"
+				(path "/eed97ac6-b1d8-4052-bc40-1c993c6f2bcf"
+					(reference "#PWR056")
+					(unit 1)
+				)
