File: carrier-orange pi zero 3w/_restore_backup_2026-09-25T20-48-06-956/EINK.kicad_sch (KiCad schematic)
At the start: 3 parts, among them J1 EPAPER_HAT_B

Commit message: ain
Parts:
- C13, C14: footprint Capacitor_SMD:C_0805_2012Metric -> (none)
Changed lines of the file:
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@@
 			)
 		)
-		(property "Footprint" "Capacitor_SMD:C_0805_2012Metric"
+		(property "Footprint" ""
 			(at 65.7352 71.12 0)
 			(hide yes)
@@
 			)
 		)
-		(property "Footprint" "Capacitor_SMD:C_0805_2012Metric"
+		(property "Footprint" ""
 			(at 78.4352 71.12 0)
 			(hide yes)
