File: carrier-orange pi zero 3w/_restore_backup_2026-09-25T20-48-06-956/USB1-7.kicad_sch (KiCad schematic)
At the start: 7 parts, among them J10 USB_A - 4, J11 USB_A - 5, J12 USB_A - 6, J13 USB_A - 7, J14 USB_A - 2, J7 USB_A - 1, J9 USB_A - 3

Commit message: ain
Parts:
- J10, J11, J7, J9: footprint USB_A_4UCON_18666_KICAD10:USB_A_4UCON_18666 -> (none)
Changed lines of the file:
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@@
 	)
 	(label "USB3DM"
-		(at 153.67 63.5 180)
+		(at 149.86 40.64 180)
 		(effects
 			(font
@@
 	)
 	(label "USB6DP"
-		(at 129.54 71.12 180)
+		(at 125.73 48.26 180)
 		(effects
 			(font
@@
 	)
 	(label "USB4DP"
-		(at 129.54 66.04 180)
+		(at 125.73 43.18 180)
 		(effects
 			(font
@@
 	)
 	(label "USB7DM"
-		(at 153.67 73.66 180)
+		(at 149.86 50.8 180)
 		(effects
 			(font
@@
 	)
 	(label "USB5DM"
-		(at 153.67 68.58 180)
+		(at 149.86 45.72 180)
 		(effects
 			(font
@@
 	)
 	(label "USB7DP"
-		(at 129.54 73.66 180)
+		(at 125.73 50.8 180)
 		(effects
 			(font
@@
 	)
 	(label "USB2DM"
-		(at 153.67 60.96 180)
+		(at 149.86 38.1 180)
 		(effects
 			(font
@@
 	)
 	(label "USB4DM"
-		(at 153.67 66.04 180)
+		(at 149.86 43.18 180)
 		(effects
 			(font
@@
 	)
 	(label "USB6DM"
-		(at 153.67 71.12 180)
+		(at 149.86 48.26 180)
 		(effects
 			(font
@@
 	)
 	(label "USB5DP"
-		(at 129.54 68.58 180)
+		(at 125.73 45.72 180)
 		(effects
 			(font
@@
 	)
 	(label "USB3DP"
-		(at 129.54 63.5 180)
+		(at 125.73 40.64 180)
 		(effects
 			(font
@@
 	)
 	(label "USB1DM"
-		(at 153.67 58.42 180)
+		(at 149.86 35.56 180)
 		(effects
 			(font
@@
 	)
 	(label "USB2DP"
-		(at 129.54 60.96 180)
+		(at 125.73 38.1 180)
 		(effects
 			(font
@@
 	)
 	(label "USB1DP"
-		(at 129.54 58.42 180)
+		(at 125.73 35.56 180)
 		(effects
 			(font
@@
 	(hierarchical_label "USBDN4_DM"
 		(shape bidirectional)
-		(at 153.67 66.04 0)
+		(at 149.86 43.18 0)
 		(effects
 			(font
@@
 	(hierarchical_label "USBDN4_DP"
 		(shape bidirectional)
-		(at 129.54 66.04 0)
+		(at 125.73 43.18 0)
 		(effects
 			(font
@@
 	(hierarchical_label "USBDN6_DM"
 		(shape bidirectional)
-		(at 153.67 71.12 0)
+		(at 149.86 48.26 0)
 		(effects
 			(font
@@
 	(hierarchical_label "USBDN5_DP"
 		(shape bidirectional)
-		(at 129.54 68.58 0)
+		(at 125.73 45.72 0)
 		(effects
 			(font
@@
 	(hierarchical_label "USBDN3_DP"
 		(shape bidirectional)
-		(at 129.54 63.5 0)
+		(at 125.73 40.64 0)
 		(effects
 			(font
@@
 	(hierarchical_label "USBDN7_DM"
 		(shape bidirectional)
-		(at 153.67 73.66 0)
+		(at 149.86 50.8 0)
 		(effects
 			(font
@@
 	(hierarchical_label "USBDN7_DP"
 		(shape bidirectional)
-		(at 129.54 73.66 0)
+		(at 125.73 50.8 0)
 		(effects
 			(font
@@
 	(hierarchical_label "USBDN3_DM"
 		(shape bidirectional)
-		(at 153.67 63.5 0)
+		(at 149.86 40.64 0)
 		(effects
 			(font
@@
 	(hierarchical_label "USBDN1_DM"
 		(shape bidirectional)
-		(at 153.67 58.42 0)
+		(at 149.86 35.56 0)
 		(effects
 			(font
@@
 	(hierarchical_label "USBDN6_DP"
 		(shape bidirectional)
-		(at 129.54 71.12 0)
+		(at 125.73 48.26 0)
 		(effects
 			(font
@@
 	(hierarchical_label "USBDN1_DP"
 		(shape bidirectional)
-		(at 129.54 58.42 0)
+		(at 125.73 35.56 0)
 		(effects
 			(font
@@
 	(hierarchical_label "USBDN2_DP"
 		(shape bidirectional)
-		(at 129.54 60.96 0)
+		(at 125.73 38.1 0)
 		(effects
 			(font
@@
 	(hierarchical_label "USBDN5_DM"
 		(shape bidirectional)
-		(at 153.67 68.58 0)
+		(at 149.86 45.72 0)
 		(effects
 			(font
@@
 	(hierarchical_label "USBDN2_DM"
 		(shape bidirectional)
-		(at 153.67 60.96 0)
+		(at 149.86 38.1 0)
 		(effects
 			(font
@@
 			)
 		)
-		(property "Footprint" "USB_A_4UCON_18666_KICAD10:USB_A_4UCON_18666"
+		(property "Footprint" ""
 			(at 76.2 69.85 0)
 			(hide yes)
@@
 			)
 		)
-		(property "Footprint" "USB_A_4UCON_18666_KICAD10:USB_A_4UCON_18666"
+		(property "Footprint" ""
 			(at 43.18 129.54 0)
 			(hide yes)
@@
 			)
 		)
-		(property "Footprint" "USB_A_4UCON_18666_KICAD10:USB_A_4UCON_18666"
+		(property "Footprint" ""
 			(at 43.18 69.85 0)
 			(hide yes)
@@
 			)
 		)
-		(property "Footprint" "USB_A_4UCON_18666_KICAD10:USB_A_4UCON_18666"
+		(property "Footprint" ""
 			(at 41.91 160.02 0)
 			(hide yes)
