File: carrier-orange pi zero 3w/_restore_backup_2026-09-25T20-48-06-956/carrier-orange pi zero 3w.kicad_pcb (KiCad board)
At the start: 2 copper layers, 68 parts, among them J10 USB_A - 4, J11 USB_A - 5, J3 Orange Pi Zero 3W - 40-Pin GP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, J4 Conn_01x04_Pin, J5 ORANGE_PI_POWER_CABLE, J6 5V_PERIPHERALS, J7 USB_A - 1, J9 USB_A - 3, Q2 2N7002, U1 TPS54302DDCT

Commit message: ain
Parts:
- removed C1, C10, C14, C15, C16, C17, C18, C20, C22, C23: 100nF, Capacitor_SMD:C_0805_2012Metric
- removed C11, C12: 22µF, Capacitor_SMD:C_1206_3216Metric
- removed C13: 10µF, Capacitor_SMD:C_0805_2012Metric
- removed C19, C21, C24, C27, C28: 1µF, Capacitor_SMD:C_0805_2012Metric
- removed C25, C26: 33pF, Capacitor_SMD:C_0805_2012Metric
- removed C8: 47pF, Capacitor_SMD:C_0805_2012Metric
- removed C9: 10µF, Capacitor_SMD:C_1206_3216Metric
- removed F2: MF-R500, Capacitor_SMD:C_1206_3216Metric
- removed J10: USB_A - 4, USB_A_4UCON_18666_KICAD10:USB_A_4UCON_18666
- removed J11: USB_A - 5, USB_A_4UCON_18666_KICAD10:USB_A_4UCON_18666
- removed J7: USB_A - 1, USB_A_4UCON_18666_KICAD10:USB_A_4UCON_18666
- removed J9: USB_A - 3, USB_A_4UCON_18666_KICAD10:USB_A_4UCON_18666
- removed R10: 10 kΩ, Resistor_SMD:R_0805_2012Metric
- removed R11, R12, R13, R14, R15, R16, R17, R18, R19, R20, R21, R22, R23, R25, R27, R28: 10k, Resistor_SMD:R_0805_2012Metric
- removed R2, R24, R26, R6, R7: 100k, Resistor_SMD:R_0805_2012Metric
- removed R3: 22.1k, Resistor_SMD:R_0805_2012Metric
- removed R4: 1M, Resistor_SMD:R_0805_2012Metric
- removed R5: 12.0k, Resistor_SMD:R_0805_2012Metric
- removed R8, R9: 5.1k, Resistor_SMD:R_0805_2012Metric
- moved J5 115.1 mm to (165.9, 41.6), turned to 90 degrees
- moved F1 109.5 mm to (152.2, 41.4)
- moved R1 104.6 mm to (166.9, 44.3), turned to 180 degrees
- moved U1 90.6 mm to (196.2, 103.5)
- moved Q2 70.5 mm to (207.4, 113.5)
- moved C3 55.8 mm to (159.7, 103.9)
- moved C2 54.7 mm to (166.9, 119.3), turned to -90 degrees
- moved C6 45.0 mm to (150.9, 116.3)
- moved C7 43.3 mm to (159.8, 110.7)
- moved C5 39.6 mm to (149.8, 122.2)
- moved C4 35.1 mm to (156.0, 119.6)
- moved J6 34.2 mm to (163.4, 117.9)
Other:
- board text added: "+5V OPI"
- board text added: "CC1"
- board text added: "CC2"
