File: carrier-orange pi zero 3w/_restore_backup_2026-09-25T20-48-06-956/power.kicad_sch (KiCad schematic)
At the start: 22 parts, among them J4 Conn_01x04_Pin, J5 ORANGE_PI_POWER_CABLE, J6 5V_PERIPHERALS, U1 TPS54302DDCT

Commit message: ain
Parts:
- C1, C10, C8: footprint Capacitor_SMD:C_0805_2012Metric -> (none)
- C11, C12, C9: footprint Capacitor_SMD:C_1206_3216Metric -> (none)
- R2, R3: footprint Resistor_SMD:R_0805_2012Metric -> (none)
Changed lines of the file:
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@@
 			)
 		)
-		(property "Footprint" "Resistor_SMD:R_0805_2012Metric"
+		(property "Footprint" ""
 			(at 205.232 110.49 90)
 			(hide yes)
@@
 			)
 		)
-		(property "Footprint" "Capacitor_SMD:C_0805_2012Metric"
+		(property "Footprint" ""
 			(at 201.6252 99.06 0)
 			(hide yes)
@@
 			)
 		)
-		(property "Footprint" "Capacitor_SMD:C_1206_3216Metric"
+		(property "Footprint" ""
 			(at 253.6952 109.22 0)
 			(hide yes)
@@
 			)
 		)
-		(property "Footprint" "Capacitor_SMD:C_1206_3216Metric"
+		(property "Footprint" ""
 			(at 253.6952 132.08 0)
 			(hide yes)
@@
 			)
 		)
-		(property "Footprint" "Capacitor_SMD:C_0805_2012Metric"
+		(property "Footprint" ""
 			(at 266.3952 109.22 0)
 			(hide yes)
@@
 			)
 		)
-		(property "Footprint" "Resistor_SMD:R_0805_2012Metric"
+		(property "Footprint" ""
 			(at 211.582 121.92 90)
 			(hide yes)
@@
 			)
 		)
-		(property "Footprint" "Capacitor_SMD:C_1206_3216Metric"
+		(property "Footprint" ""
 			(at 266.3952 132.08 0)
 			(hide yes)
@@
 			)
 		)
-		(property "Footprint" "Capacitor_SMD:C_0805_2012Metric"
+		(property "Footprint" ""
 			(at 220.6752 114.3 0)
 			(hide yes)
