File: carrier-orange pi zero 3w/_restore_backup_2026-09-26T11-09-31-632/carrier-orange pi zero 3w.kicad_pcb (KiCad board)
At the start: 2 copper layers, 68 parts, among them J10 USB_A - 4, J11 USB_A - 5, J3 Orange Pi Zero 3W - 40-Pin GP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, J4 Conn_01x04_Pin, J5 ORANGE_PI_POWER_CABLE, J6 5V_PERIPHERALS, J7 USB_A - 1, J9 USB_A - 3, Q2 2N7002, U1 TPS54302DDCT

Commit message: ain
Parts:
- removed J10: USB_A - 4, USB_A_4UCON_18666_KICAD10:USB_A_4UCON_18666
- removed J11: USB_A - 5, USB_A_4UCON_18666_KICAD10:USB_A_4UCON_18666
- removed J7: USB_A - 1, USB_A_4UCON_18666_KICAD10:USB_A_4UCON_18666
- removed J9: USB_A - 3, USB_A_4UCON_18666_KICAD10:USB_A_4UCON_18666
