File: keyboard pcb/Keyboard-Doomsdaydeck.kicad_pcb (KiCad board)
At the start: 2 copper layers, 194.5 x 130.5 mm, 106 parts, among them J1 Conn_01x05, J2 Conn_01x02, J3 Conn_01x02, J4 OLED, J5 Conn_01x04_Pin, U1 Raspberry_Pi_Pico2

Commit message: ain
Routing:
- net GND: track 244.0 -> 366.4 mm
- net COL10: track 120.5 -> 242.6 mm, vias 0 -> 2
- net COL8: track 112.5 -> 194.7 mm, vias 0 -> 3
- net COL6: track 117.9 -> 179.6 mm, vias 0 -> 3
- net COL7: track 170.1 -> 178.7 mm
- net COL2: track 180.3 -> 187.8 mm
- net COL3: track 152.0 -> 156.4 mm
- net COL9: track 208.6 -> 212.1 mm
- net COL5: track 125.1 -> 128.2 mm
- net COL1: track 204.4 -> 207.5 mm
- net SDA: track 244.0 -> 245.3 mm
- net JOY_X: track 215.7 -> 216.9 mm
- net COL4: track 128.1 -> 129.2 mm, vias 2 -> 1
- net SCL: track 238.2 -> 238.8 mm
- net JOY_Y: track 110.2 -> 110.7 mm, vias 3 -> 1

Commit message: ain
Other:
- board size 194.5 x 130.5 mm -> 189.5 x 130 mm
Changed lines of the file:
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@@
 	)
 	(gr_rect
-		(start 16 40.5)
+		(start 21 41)
 		(end 210.499999 171)
 		(stroke
