File: PCB'S/CARRIER BOARD PCB/carrier-orange pi zero 3w.kicad_pcb (KiCad board)
At the start: 4 copper layers, 190 x 61 mm, 112 parts, among them J1 EPAPER_HAT_B, J10 USB_A - 4, J11 USB_A - 5, J12 USB_A - 6 (For Display), J13 USB_A - 7 (For RTL SDR), J14 USB_A - 2 (Extra/For phone ), J15 FAN1, J16 FAN2, J17 L-SPEAKER, J18 R-SPEAKER, J19 EXT-GPIO (BACKUP), J2 CORE1262_HF, J3 Orange Pi Zero 3W - 40-Pin GP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, J4 Conn_01x04_Pin, J5 EXT-GPIO, J6 PWR FOR DISPLAY, J7 USB_A - 1, J8 Usb-C receptable, J9 USB_A - 3, Q1 Q_PMOS_GSD, Q2 2N7002, Q3 AO3400A, Q4 AO3400A, U1 TPS54302DDCT, U2 USB2517I-JZX, U3 TPD2EUSB30DRTR, U4 L-MAX98357AETE+T, U5 R-MAX98357AETE+T, U7 MCP23017x-x-SO, Y1 24.000MHz

Commit message: ain
Routing:
- net GND: track 117.0 -> 118.9 mm
Changed lines of the file:
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@@
 	)
 	(segment
+		(start 157.96 44.29)
+		(end 130.7 44.29)
+		(width 0.8)
+		(layer "F.Cu")
+		(net "+5V_USB")
+	)
+	(segment
+		(start 130.7 44.29)
+		(end 129.58 45.41)
+		(width 0.8)
+		(layer "F.Cu")
+		(net "+5V_USB")
+	)
+	(segment
 		(start 81.28 65.05)
 		(end 80.61 65.72)
@@
 	)
 	(segment
+		(start 160.03 58.68)
+		(end 160.03 46.36)
+		(width 0.8)
+		(layer "F.Cu")
+		(net "+5V_USB")
+	)
+	(segment
 		(start 102.46 45.41)
 		(end 98.94 45.41)
@@
 	)
 	(segment
-		(start 160.03 56.85)
-		(end 160.03 46.36)
-		(width 0.8)
-		(layer "F.Cu")
-		(net "+5V_USB")
-	)
-	(segment
 		(start 112.9 44.65)
 		(end 112.9 41.4)
@@
 	)
 	(segment
-		(start 174.884879 71.704879)
-		(end 160.03 56.85)
-		(width 0.8)
-		(layer "F.Cu")
-		(net "+5V_USB")
-	)
-	(segment
-		(start 157.96 44.29)
-		(end 130.7 44.29)
-		(width 0.8)
-		(layer "F.Cu")
-		(net "+5V_USB")
-	)
-	(segment
-		(start 174.884879 74.5)
-		(end 174.884879 71.704879)
+		(start 174.884879 73.534879)
+		(end 160.03 58.68)
 		(width 0.8)
 		(layer "F.Cu")
@@
 	)
 	(segment
+		(start 174.884879 74.5)
+		(end 174.884879 73.534879)
+		(width 0.8)
+		(layer "F.Cu")
+		(net "+5V_USB")
+	)
+	(segment
 		(start 129.965 44.29)
 		(end 137.952692 44.29)
@@
 	)
 	(segment
-		(start 130.7 44.29)
-		(end 129.58 45.41)
-		(width 0.8)
-		(layer "F.Cu")
-		(net "+5V_USB")
-	)
-	(segment
 		(start 137.952692 44.29)
 		(end 146.462692 35.78)
@@
 	)
 	(segment
+		(start 236.35 54.75)
+		(end 235.65 54.75)
+		(width 0.2)
+		(layer "F.Cu")
+		(net "GND")
+	)
+	(segment
 		(start 179.76 66.515)
 		(end 181.4 64.875)
@@
 	)
 	(segment
-		(start 235.65 54.75)
-		(end 236.64 54.75)
-		(width 0.2)
-		(layer "F.Cu")
-		(net "GND")
-	)
-	(segment
 		(start 173.422379 83.945)
 		(end 174.525 83.945)
@@
 	)
 	(segment
-		(start 110.55 64.95)
-		(end 110.55 66.72)
+		(start 236.5 54.6)
+		(end 236.35 54.75)
 		(width 0.2)
 		(layer "F.Cu")
@@
 	)
 	(segment
-		(start 236.64 54.75)
-		(end 236.69 54.8)
+		(start 110.55 64.95)
+		(end 110.55 66.72)
 		(width 0.2)
 		(layer "F.Cu")
@@
 	)
 	(segment
+		(start 236.5 52.55)
+		(end 236.5 54.6)
+		(width 0.2)
+		(layer "F.Cu")
+		(net "GND")
+	)
+	(segment
 		(start 104.84 39.85)
 		(end 104.84 41.39)
@@
 	)
 	(via
-		(at 236.69 54.8)
+		(at 236.5 52.55)
 		(size 0.6)
 		(drill 0.3)
@@
 	)
 	(segment
-		(start 238.4 54.2)
-		(end 237.2 55.4)
-		(width 0.2)
-		(layer "F.Cu")
-		(net "Net-(J18-Pin_2)")
-	)
-	(segment
-		(start 236.291471 55.25)
+		(start 237.35 55.25)
 		(end 235.65 55.25)
 		(width 0.2)
@@
 	)
 	(segment
-		(start 245.95 54.2)
-		(end 238.4 54.2)
-		(width 0.2)
-		(layer "F.Cu")
-		(net "Net-(J18-Pin_2)")
-	)
-	(segment
-		(start 237.2 55.4)
-		(end 236.441471 55.4)
+		(start 247.6 55.85)
+		(end 245.55 53.8)
 		(width 0.2)
 		(layer "F.Cu")
@@
 	)
 	(segment
-		(start 247.6 55.85)
-		(end 245.95 54.2)
+		(start 238.8 53.8)
+		(end 237.35 55.25)
 		(width 0.2)
 		(layer "F.Cu")
@@
 	)
 	(segment
-		(start 236.441471 55.4)
-		(end 236.291471 55.25)
+		(start 245.55 53.8)
+		(end 238.8 53.8)
 		(width 0.2)
 		(layer "F.Cu")
