File: PCB'S/CARRIER BOARD PCB/USB.kicad_sch (KiCad schematic)
At the start: 44 parts, among them J8 Usb-C receptable, Q1 Q_PMOS_GSD, Q2 2N7002, U2 USB2517I-JZX, U3 TPD2EUSB30DRTR, Y1 24.000MHz

Commit message: ain
Other:
- moved on the sheet: C15, C22, C24, C28
Changed lines of the file:
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@@
 	)
 	(rectangle
-		(start 53.975 171.45)
-		(end 110.49 196.85)
+		(start 15.875 207.01)
+		(end 72.39 232.41)
 		(stroke
 			(width 0)
@@
 	)
 	(junction
-		(at 93.98 181.61)
+		(at 55.88 217.17)
 		(diameter 0)
 		(color 0 0 0 0)
 	)
 	(junction
-		(at 68.58 181.61)
+		(at 30.48 217.17)
 		(diameter 0)
 		(color 0 0 0 0)
@@
 	(wire
 		(pts
-			(xy 68.58 175.26) (xy 68.58 181.61)
+			(xy 30.48 210.82) (xy 30.48 217.17)
 		)
 		(stroke
@@
 	(wire
 		(pts
-			(xy 68.58 181.61) (xy 68.58 189.23)
+			(xy 30.48 217.17) (xy 30.48 224.79)
 		)
 		(stroke
@@
 	(wire
 		(pts
-			(xy 93.98 173.99) (xy 93.98 181.61)
+			(xy 55.88 209.55) (xy 55.88 217.17)
 		)
 		(stroke
@@
 	(wire
 		(pts
-			(xy 93.98 181.61) (xy 93.98 190.5)
+			(xy 55.88 217.17) (xy 55.88 226.06)
 		)
 		(stroke
@@
 	)
 	(label "VDDA33_1"
-		(at 68.58 175.26 0)
+		(at 30.48 210.82 0)
 		(effects
 			(font
@@
 	)
 	(label "VDD33CR"
-		(at 93.98 173.99 0)
+		(at 55.88 209.55 0)
 		(effects
 			(font
@@
 	(global_label "+3V3_MAIN"
 		(shape input)
-		(at 68.58 176.53 180)
+		(at 30.48 212.09 180)
 		(fields_autoplaced yes)
 		(effects
@@
 		)
 		(property "Intersheetrefs" "${INTERSHEET_REFS}"
-			(at 55.0719 176.53 0)
+			(at 16.9719 212.09 0)
 			(hide yes)
 			(show_name no)
@@
 	(global_label "+3V3_MAIN"
 		(shape input)
-		(at 93.98 176.53 180)
+		(at 55.88 212.09 180)
 		(fields_autoplaced yes)
 		(effects
@@
 		)
 		(property "Intersheetrefs" "${INTERSHEET_REFS}"
-			(at 80.4719 176.53 0)
+			(at 42.3719 212.09 0)
 			(hide yes)
 			(show_name no)
@@
 	(symbol
 		(lib_id "Device:C")
-		(at 72.39 189.23 90)
+		(at 34.29 224.79 90)
 		(unit 1)
 		(body_style 1)
@@
 		(dnp no)
 		(property "Reference" "C28"
-			(at 73.66 192.024 90)
+			(at 35.56 227.584 90)
 			(show_name no)
 			(do_not_autoplace no)
@@
 		)
 		(property "Value" "1µF"
-			(at 74.422 186.69 90)
+			(at 36.322 222.25 90)
 			(show_name no)
 			(do_not_autoplace no)
@@
 		)
 		(property "Footprint" "Capacitor_SMD:C_0805_2012Metric"
-			(at 76.2 188.2648 0)
+			(at 38.1 223.8248 0)
 			(hide yes)
 			(show_name no)
@@
 		)
 		(property "Datasheet" ""
-			(at 72.39 189.23 0)
+			(at 34.29 224.79 0)
 			(hide yes)
 			(show_name no)
@@
 		)
 		(property "Description" "Unpolarized capacitor"
-			(at 72.39 189.23 0)
+			(at 34.29 224.79 0)
 			(hide yes)
 			(show_name no)
@@
 	(symbol
 		(lib_id "Device:C")
-		(at 72.39 181.61 90)
+		(at 34.29 217.17 90)
 		(unit 1)
 		(body_style 1)
@@
 		(dnp no)
 		(property "Reference" "C15"
-			(at 72.39 184.912 90)
+			(at 34.29 220.472 90)
 			(show_name no)
 			(do_not_autoplace no)
@@
 		)
 		(property "Value" "100nF"
-			(at 72.898 178.562 90)
+			(at 34.798 214.122 90)
 			(show_name no)
 			(do_not_autoplace no)
@@
 		)
 		(property "Footprint" "Capacitor_SMD:C_0805_2012Metric"
-			(at 76.2 180.6448 0)
+			(at 38.1 216.2048 0)
 			(hide yes)
 			(show_name no)
@@
 		)
 		(property "Datasheet" ""
-			(at 72.39 181.61 0)
+			(at 34.29 217.17 0)
 			(hide yes)
 			(show_name no)
@@
 		)
 		(property "Description" "Unpolarized capacitor"
-			(at 72.39 181.61 0)
+			(at 34.29 217.17 0)
 			(hide yes)
 			(show_name no)
@@
 	(symbol
 		(lib_id "power:GND")
-		(at 101.6 181.61 0)
+		(at 63.5 217.17 0)
 		(unit 1)
 		(body_style 1)
@@
 		(dnp no)
 		(property "Reference" "#PWR026"
-			(at 101.6 187.96 0)
+			(at 63.5 223.52 0)
 			(hide yes)
 			(show_name no)
@@
 		)
 		(property "Value" "GND"
-			(at 105.156 183.388 0)
+			(at 67.056 218.948 0)
 			(show_name no)
 			(do_not_autoplace no)
@@
 		)
 		(property "Footprint" ""
-			(at 101.6 181.61 0)
+			(at 63.5 217.17 0)
 			(hide yes)
 			(show_name no)
@@
 		)
 		(property "Datasheet" ""
-			(at 101.6 181.61 0)
+			(at 63.5 217.17 0)
 			(hide yes)
 			(show_name no)
@@
 		)
 		(property "Description" "Power symbol creates a global label with name \"GND\" , ground"
-			(at 101.6 181.61 0)
+			(at 63.5 217.17 0)
 			(hide yes)
 			(show_name no)
@@
 	(symbol
 		(lib_id "Device:C")
-		(at 97.79 181.61 90)
+		(at 59.69 217.17 90)
 		(unit 1)
 		(body_style 1)
@@
 		(dnp no)
 		(property "Reference" "C24"
-			(at 99.314 184.912 90)
+			(at 61.214 220.472 90)
 			(show_name no)
 			(do_not_autoplace no)
@@
 		)
 		(property "Value" "1µF"
-			(at 101.092 178.816 90)
+			(at 62.992 214.376 90)
 			(show_name no)
 			(do_not_autoplace no)
@@
 		)
 		(property "Footprint" "Capacitor_SMD:C_0805_2012Metric"
-			(at 101.6 180.6448 0)
+			(at 63.5 216.2048 0)
 			(hide yes)
 			(show_name no)
@@
 		)
 		(property "Datasheet" ""
-			(at 97.79 181.61 0)
+			(at 59.69 217.17 0)
 			(hide yes)
 			(show_name no)
@@
 		)
 		(property "Description" "Unpolarized capacitor"
-			(at 97.79 181.61 0)
+			(at 59.69 217.17 0)
 			(hide yes)
 			(show_name no)
@@
 	(symbol
 		(lib_id "power:GND")
-		(at 76.2 189.23 0)
+		(at 38.1 224.79 0)
 		(unit 1)
 		(body_style 1)
@@
 		(dnp no)
 		(property "Reference" "#PWR031"
-			(at 76.2 195.58 0)
+			(at 38.1 231.14 0)
 			(hide yes)
 			(show_name no)
@@
 		)
 		(property "Value" "GND"
-			(at 78.232 191.516 0)
+			(at 40.132 227.076 0)
 			(show_name no)
 			(do_not_autoplace no)
@@
 		)
 		(property "Footprint" ""
-			(at 76.2 189.23 0)
+			(at 38.1 224.79 0)
 			(hide yes)
 			(show_name no)
@@
 		)
 		(property "Datasheet" ""
-			(at 76.2 189.23 0)
+			(at 38.1 224.79 0)
 			(hide yes)
 			(show_name no)
@@
 		)
 		(property "Description" "Power symbol creates a global label with name \"GND\" , ground"
-			(at 76.2 189.23 0)
+			(at 38.1 224.79 0)
 			(hide yes)
 			(show_name no)
@@
 	(symbol
 		(lib_id "power:GND")
-		(at 76.2 181.61 0)
+		(at 38.1 217.17 0)
 		(unit 1)
 		(body_style 1)
@@
 		(dnp no)
 		(property "Reference" "#PWR019"
-			(at 76.2 187.96 0)
+			(at 38.1 223.52 0)
 			(hide yes)
 			(show_name no)
@@
 		)
 		(property "Value" "GND"
-			(at 78.232 182.118 0)
+			(at 40.132 217.678 0)
 			(show_name no)
 			(do_not_autoplace no)
@@
 		)
 		(property "Footprint" ""
-			(at 76.2 181.61 0)
+			(at 38.1 217.17 0)
 			(hide yes)
 			(show_name no)
@@
 		)
 		(property "Datasheet" ""
-			(at 76.2 181.61 0)
+			(at 38.1 217.17 0)
 			(hide yes)
 			(show_name no)
@@
 		)
 		(property "Description" "Power symbol creates a global label with name \"GND\" , ground"
-			(at 76.2 181.61 0)
+			(at 38.1 217.17 0)
 			(hide yes)
 			(show_name no)
@@
 	(symbol
 		(lib_id "Device:C")
-		(at 97.79 190.5 90)
+		(at 59.69 226.06 90)
 		(unit 1)
 		(body_style 1)
@@
 		(dnp no)
 		(property "Reference" "C22"
-			(at 98.806 194.056 90)
+			(at 60.706 229.616 90)
 			(show_name no)
 			(do_not_autoplace no)
@@
 		)
 		(property "Value" "100nF"
-			(at 102.108 187.452 90)
+			(at 64.008 223.012 90)
 			(show_name no)
 			(do_not_autoplace no)
@@
 		)
 		(property "Footprint" "Capacitor_SMD:C_0805_2012Metric"
-			(at 101.6 189.5348 0)
+			(at 63.5 225.0948 0)
 			(hide yes)
 			(show_name no)
@@
 		)
 		(property "Datasheet" ""
-			(at 97.79 190.5 0)
+			(at 59.69 226.06 0)
 			(hide yes)
 			(show_name no)
@@
 		)
 		(property "Description" "Unpolarized capacitor"
-			(at 97.79 190.5 0)
+			(at 59.69 226.06 0)
 			(hide yes)
 			(show_name no)
@@
 	(symbol
 		(lib_id "power:GND")
-		(at 101.6 190.5 0)
+		(at 63.5 226.06 0)
 		(unit 1)
 		(body_style 1)
@@
 		(dnp no)
 		(property "Reference" "#PWR023"
-			(at 101.6 196.85 0)
+			(at 63.5 232.41 0)
 			(hide yes)
 			(show_name no)
@@
 		)
 		(property "Value" "GND"
-			(at 105.156 192.278 0)
+			(at 67.056 227.838 0)
 			(show_name no)
 			(do_not_autoplace no)
@@
 		)
 		(property "Footprint" ""
-			(at 101.6 190.5 0)
+			(at 63.5 226.06 0)
 			(hide yes)
 			(show_name no)
@@
 		)
 		(property "Datasheet" ""
-			(at 101.6 190.5 0)
+			(at 63.5 226.06 0)
 			(hide yes)
 			(show_name no)
@@
 		)
 		(property "Description" "Power symbol creates a global label with name \"GND\" , ground"
-			(at 101.6 190.5 0)
+			(at 63.5 226.06 0)
 			(hide yes)
 			(show_name no)
