File: PCB'S/KEYBOARD'S PCB/Keyboard-Doomsdaydeck.kicad_pcb (KiCad board)
At the start: 2 copper layers, 189.5 x 130 mm, 106 parts, among them J1 Conn_01x05, J2 Conn_01x02, J3 Conn_01x02, J4 OLED, J5 Conn_01x04_Pin, U1 Raspberry_Pi_Pico2

Commit message: ain
Parts:
- added J6: Conn_01x04_Pin, Connector:FanPinHeader_1x04_P2.54mm_Vertical, F.Cu at (193.0, 156.7)
Connections:
- J5 pad 2: unconnected-(J5-Pin_2-Pad2) -> 5V
- J5 pad 3: SDA -> unconnected-(J5-Pin_3-Pad3)
- J5 pad 4: SCL -> unconnected-(J5-Pin_4-Pad4)
Routing:
- net 5V: track 0.00 -> 108.2 mm
- net GND: track 366.4 -> 456.5 mm, vias 0 -> 2
- net SDA: track 245.3 -> 267.9 mm
- net SCL: track 238.8 -> 257.4 mm, vias 2 -> 4
- net COL10: track 242.6 -> 243.4 mm
